File: hardware/a1200-psu/a1200-psu.kicad_sch (KiCad schematic)
At the start: 59 parts, among them J1 220V, J2 Conn_01x05, Q1 P2N60, SW1 SW_SPST, U1 UC3844_DIP8, U2 PC817, U3 TL431D

Commit message: Fixed R values and added to PCB
Parts:
- removed C12: 68n, symbol Device:C_Small
- removed D2: ?, symbol Device:D
- added C12: 47uF, Capacitor_THT:CP_Radial_D6.3mm_P2.50mm, symbol a500-psu-rescue:CP1_Small-Device
- added C20: 1nF, Capacitor_THT:C_Rect_L7.0mm_W2.5mm_P5.00mm, symbol Device:C_Small
- added C21: 470pF, Capacitor_THT:C_Rect_L7.0mm_W4.5mm_P5.00mm, symbol Device:C_Small
- added D2: 1N4742A, Diode_THT:D_DO-35_SOD27_P10.16mm_Horizontal, symbol Device:D_Zener
- C1: value 10n -> 10nF; footprint (none) -> Capacitor_THT:C_Rect_L7.0mm_W2.5mm_P5.00mm
- C10: footprint (none) -> Capacitor_THT:C_Disc_D9.0mm_W5.0mm_P10.00mm
- C11: value 33u -> 33uF; footprint (none) -> Capacitor_THT:C_Radial_D16.0mm_H31.5mm_P7.50mm
- C4: value 47u -> 10nF; footprint (none) -> Capacitor_THT:C_Rect_L7.0mm_W2.5mm_P5.00mm
- C9: value ? -> 220pF; footprint (none) -> Capacitor_THT:C_Disc_D6.0mm_W2.5mm_P5.00mm
- D1: value ? -> 1N4007; footprint (none) -> Diode_THT:D_DO-41_SOD81_P10.16mm_Horizontal; VR (none) -> 1000V
- D10, D9: value GI850 -> MR852
- D3: value ? -> BYV26E; footprint (none) -> Diode_THT:D_DO-41_SOD81_P7.62mm_Horizontal
- D4: VR (none) -> 1000V
- D5: value 1N49** -> 1N4935; VR (none) -> 200V
- D7: value FR107 -> 1N54xx
- D8: value SPR50 -> MR852
- F1: value 250V 1A FIA -> 250V T 1A
- L1: footprint (none) -> Filter:Filter_FILTERCON_1FPxx
- Q1: footprint Package_TO_SOT_THT:TO-220-3_Vertical -> Amiga 1200:TO-220-3_Vertical_Staggered
- R1: value ? -> 680R; footprint (none) -> Resistor_THT:R_Axial_DIN0207_L6.3mm_D2.5mm_P10.16mm_Horizontal
- R10, R7: footprint (none) -> Resistor_THT:R_Axial_DIN0309_L9.0mm_D3.2mm_P12.70mm_Horizontal
- R11, R8: footprint (none) -> Resistor_THT:R_Axial_DIN0207_L6.3mm_D2.5mm_P10.16mm_Horizontal
- R2: value 23k? -> 240k; footprint (none) -> Resistor_THT:R_Axial_DIN0207_L6.3mm_D2.5mm_P10.16mm_Horizontal
- R3: value 23k? -> 25k5; footprint (none) -> Resistor_THT:R_Axial_DIN0207_L6.3mm_D2.5mm_P10.16mm_Horizontal
- R4: value ? -> 821k; footprint (none) -> Resistor_THT:R_Axial_DIN0309_L9.0mm_D3.2mm_P12.70mm_Horizontal
- R5: footprint (none) -> Resistor_THT:R_Axial_DIN0309_L9.0mm_D3.2mm_P15.24mm_Horizontal
- R6: value 1M? -> 460R; footprint (none) -> Resistor_THT:R_Axial_DIN0207_L6.3mm_D2.5mm_P10.16mm_Horizontal
- R9: value 1R2? -> 1R; footprint (none) -> Resistor_THT:R_Axial_DIN0309_L9.0mm_D3.2mm_P12.70mm_Horizontal
- U3: footprint Package_SO:SOIC-8_3.9x4.9mm_P1.27mm -> Package_TO_SOT_THT:TO-92L
Connections:
- net +12VA: now also C12.1; no longer C4.2
- net +5V: now also J2.3 (Red); no longer J2.4 (Red)
- net GND: now also J2.4 (Black); no longer J2.3 (Black)
- net GNDD: now also C1.1, C12.2, C20.1, C21.2, D2.2 (A); no longer C4.1, R4.2
- net at R2.2, R3.2, U1.4 (RC): now also C4.2, C20.2; no longer C1.2
- net at C10.1, C11.1, D4.1 (+)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: now also R4.1; no longer R6.1
- net at R1.2, U1.1 (COMP), U2.4: now also C1.2, C4.1; no longer C1.1
- net at C9.1, Q1.3 (S), R9.1: now also R6.2, D2.1 (K)
- new net: C21.1, R4.2, R6.1, U1.3 (CS)
Other:
- note added: "100R OK?"
- note added: "16 V"
- note added: "1M OK?"
- note added: "340 V"
- note added: "470R OK?"
- note added: "All caps and diodes on stepped down side should be correct for A1200"
- note added: "Based on the A500 PSU schematic by Greg McCarthy (https://github.com/StormTrooper) Some part values will still be for A500 PSU, so always double check before ordering"
- note added: "Line filter"
- note added: "Main cap 400ms to charge to 334 V 1.2s to discharge to 18 V"
- note added: "Test of known good working UC3844 PWM IC Pin 6 (OUT) Load on 5V output I (5 V) | Duty | Period | V max ---- | ----- | ---- | ---- 0 mA | 7.0% | 276 ms | 18.0 V 28 mA | 4.0% | 25 us | 12.2 V 1.0 A | 9.5% | 25 us | 14.8 V 3.0 A | 15.0% | 25 us | 16.4 V 6.0 A | 20.0% | 25 us | 19.0 V"
- note removed: "Based on the A500 PSU schematic by Greg McCarthy (https://github.com/StormTrooper)"
- note removed: "TODO: Cap at FET pin 2"
- note removed: "TODO: Check if diode (light grey)"
- note removed: "TODO: How does this not zap IC with 240V?"
- note removed: "TODO: Small blue block"
- note removed: "TODO: White bulb, diode?"
- note removed: "Test of known good working UC3844 PWM IC Pin 6 (OUT) Load on 5V output I | Duty | Period | V max ---- | ----- | ---- | ---- 0 mA | 7.0% | 276 ms | 18.0 V 28 mA | 4.0% | 25 us | 12.2 V 1.0 A | 9.5% | 25 us | 14.8 V 3.0 A | 15.0% | 25 us | 16.4 V 6.0 A | 20.0% | 25 us | 19.0 V"
- moved on the sheet: C13, C14, C15, C16, C17, C18, C19, C9, D1, D10, D5, D7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

Commit message: Add transformer footprint
Parts:
- TR1: footprint Transformer_THT:Transformer_CHK_EI48-8VA_Neutral -> Amiga 1200:Transformer
Changed lines of the file:
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@@
       (effects (font (size 1.27 1.27)) hide)
     )
-    (property "Footprint" "Transformer_THT:Transformer_CHK_EI48-8VA_Neutral" (id 2) (at 219.71 139.7 0)
+    (property "Footprint" "Amiga 1200:Transformer" (id 2) (at 219.71 139.7 0)
       (effects (font (size 1.27 1.27)) hide)
     )
@@
     )
     (path "/32bac948-60ce-4bc5-be71-ae7e97ee9e18"
-      (reference "TR1") (unit 1) (value "A1200-PSU-TR") (footprint "Transformer_THT:Transformer_CHK_EI48-8VA_Neutral")
+      (reference "TR1") (unit 1) (value "A1200-PSU-TR") (footprint "Amiga 1200:Transformer")
     )
     (path "/ce52b9e9-9f67-4642-b228-ee4173e43849"
