File: hardware/a1200-psu/a1200-psu.kicad_pcb (KiCad board)
At the start: 2 copper layers, 147 x 76 mm, 61 parts, among them J1 AC-In, J2 DC-Out, Q1 P2N60, U1 UC3844_DIP8, U2 PC817, U3 TL431D

Commit message: Reorganised PWM IC power supply
Also discovered some new part values
Parts:
- added D11: Yellow, LED_THT:LED_D3.0mm, F.Cu at (90.2, 31.2)
- added R18: 500k, Resistor_THT:R_Axial_DIN0207_L6.3mm_D2.5mm_P10.16mm_Horizontal, F.Cu at (95.2, 31.2)
- D6: value ? -> 1N5230B
- moved R1 10.2 mm to (111.3, 83.8), turned to -90 degrees
Connections:
- net +12VA renamed Net-(R5-Pad1)
- net Net-(C10-Pad1) renamed +330V
- net Net-(R11-Pad2) renamed /TR1_P5
- R1 pad 1: Net-(R1-Pad1) -> Net-(C1-Pad2)
- R1 pad 2: Net-(C1-Pad2) -> Net-(R2-Pad1)
- R2 pad 1: Net-(R1-Pad1) -> Net-(R2-Pad1)
- R3 pad 1: Net-(R1-Pad1) -> Net-(R2-Pad1)
- U1 pad 8: Net-(R1-Pad1) -> Net-(R2-Pad1)
Routing:
- net +330V: track 99.9 -> 128.1 mm, vias 0 -> 1
- net Net-(R2-Pad1): track 0.00 -> 23.4 mm
- net Net-(R1-Pad1): track 23.4 -> 0.00 mm
- net GNDD: track 246.3 -> 249.9 mm
- net Net-(D11-Pad2): track 0.00 -> 2.55 mm
- net Net-(C1-Pad2): track 44.8 -> 44.3 mm
Other:
- outline, holes or cut-outs redrawn
- board text added: "Measurements not accurate"
