File: hardware/cpc1-psu/cpc1-psu.kicad_pcb (KiCad board)
At the start: 2 copper layers, 13 parts

Commit message: Changed part number
Parts:
- C3, C4: value 220uF 16V -> 2200uF 16V
- C5, C6: value 110uF 16V -> 100uF 16V
Changed lines of the file:
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@@
         (effects (font (size 1 1) (thickness 0.15)))
     )
-    (fp_text value "110uF 16V" (at 2.5 7.5) (layer "F.Fab")
+    (fp_text value "100uF 16V" (at 2.5 7.5) (layer "F.Fab")
         (effects (font (size 1 1) (thickness 0.15)))
     )
@@
     (descr "CP, Radial series, Radial, pin pitch=7.50mm, , diameter=18mm, Electrolytic Capacitor")
     (tags "CP Radial series Radial pin pitch 7.50mm  diameter 18mm Electrolytic Capacitor")
-    (property "Farnell" "2841894")
+    (property "Farnell" "2508122")
     (property "Sheetfile" "cpc1-psu.kicad_sch")
     (property "Sheetname" "")
@@
         (effects (font (size 1 1) (thickness 0.15)))
     )
-    (fp_text value "220uF 16V" (at 3.75 10.25 90) (layer "F.Fab")
+    (fp_text value "2200uF 16V" (at 3.75 10.25 90) (layer "F.Fab")
         (effects (font (size 1 1) (thickness 0.15)))
     )
@@
     (descr "CP, Radial series, Radial, pin pitch=7.50mm, , diameter=18mm, Electrolytic Capacitor")
     (tags "CP Radial series Radial pin pitch 7.50mm  diameter 18mm Electrolytic Capacitor")
-    (property "Farnell" "2841894")
+    (property "Farnell" "2508122")
     (property "Sheetfile" "cpc1-psu.kicad_sch")
     (property "Sheetname" "")
@@
         (effects (font (size 1 1) (thickness 0.15)))
     )
-    (fp_text value "220uF 16V" (at 3.75 10.25 90) (layer "F.Fab")
+    (fp_text value "2200uF 16V" (at 3.75 10.25 90) (layer "F.Fab")
         (effects (font (size 1 1) (thickness 0.15)))
     )
@@
     (descr "CP, Radial series, Radial, pin pitch=2.00mm, , diameter=5mm, Electrolytic Capacitor")
     (tags "CP Radial series Radial pin pitch 2.00mm  diameter 5mm Electrolytic Capacitor")
-    (property "Farnell" "")
+    (property "Farnell" "2217568")
     (property "Sheetfile" "cpc1-psu.kicad_sch")
     (property "Sheetname" "")
@@
         (effects (font (size 1 1) (thickness 0.15)))
     )
-    (fp_text value "110uF 16V" (at 2.5 7.5 90) (layer "F.Fab")
+    (fp_text value "100uF 16V" (at 2.5 7.5 90) (layer "F.Fab")
         (effects (font (size 1 1) (thickness 0.15)))
     )
@@
     (descr "CP, Radial series, Radial, pin pitch=2.00mm, , diameter=5mm, Electrolytic Capacitor")
     (tags "CP Radial series Radial pin pitch 2.00mm  diameter 5mm Electrolytic Capacitor")
-    (property "Farnell" "")
+    (property "Farnell" "2805620")
     (property "Sheetfile" "cpc1-psu.kicad_sch")
     (property "Sheetname" "")
@@
     (descr "CP, Radial series, Radial, pin pitch=2.00mm, , diameter=5mm, Electrolytic Capacitor")
     (tags "CP Radial series Radial pin pitch 2.00mm  diameter 5mm Electrolytic Capacitor")
-    (property "Farnell" "")
+    (property "Farnell" "2217568")
     (property "Sheetfile" "cpc1-psu.kicad_sch")
     (property "Sheetname" "")
